File: hardware/gnss.kicad_sch (KiCad schematic)
At the start: 11 parts, among them U1 SAM-M10Q

Commit message: beginnings of power distribution maybe?
Parts:
- added C10: 22u, symbol Device:C
- added C11: 0.1u, symbol Device:C
Connections:
- net +3V3: now also C10.1, C11.1
- net GND: now also C10.2, C11.2
Other:
- note removed: "https://github.com/sparkfun/SparkFun_u-blox_SAM-M10Q"
- note removed: "https://github.com/sparkfun/SparkFun_u-blox_SAM-M10Q/blob/main/Documentation/SAM-M10Q_DataSheet_UBX-22013293.pdf"
